Commit message: 250218_

File: exts/humarconoid/humarconoid/robots/G1/g1_29dof_rev_1_0.urdf (robot description, URDF)
Before this commit: robot g1_kist, 39 links, 38 joints
Links:
- link left_knee_link: geometry collision mesh filename=meshes_kist/left_knee_link.STL; visual mesh filename=meshes_kist/left_knee_link.STL
- link left_rubber_hand: geometry collision mesh filename=meshes_kist/left_rubber_hand.STL; visual mesh filename=meshes_kist/left_rubber_hand.STL
- link right_knee_link: geometry collision mesh filename=meshes_kist/right_knee_link.STL; visual mesh filename=meshes_kist/right_knee_link.STL
- link right_rubber_hand: geometry collision mesh filename=meshes_kist/right_rubber_hand.STL; visual mesh filename=meshes_kist/right_rubber_hand.STL
Joints:
- joint left_elbow_joint: type revolute -> fixed
- joint left_shoulder_pitch_joint: type revolute -> fixed
- joint left_shoulder_yaw_joint: type revolute -> fixed
- joint left_wrist_pitch_joint: type revolute -> fixed
- joint left_wrist_roll_joint: type revolute -> fixed
- joint left_wrist_yaw_joint: type revolute -> fixed
- joint right_elbow_joint: type revolute -> fixed
- joint right_shoulder_pitch_joint: type revolute -> fixed
- joint right_shoulder_yaw_joint: type revolute -> fixed
- joint right_wrist_pitch_joint: type revolute -> fixed
- joint right_wrist_roll_joint: type revolute -> fixed
- joint right_wrist_yaw_joint: type revolute -> fixed

Commit message: 250221

File: exts/humarconoid/humarconoid/robots/G1/g1_29dof_rev_1_0.urdf (robot description, URDF)
Before this commit: robot g1_kist, 39 links, 38 joints
Joints:
- joint left_shoulder_roll_joint: type revolute -> fixed
- joint right_shoulder_roll_joint: type revolute -> fixed
- joint waist_pitch_joint: type revolute -> fixed
- joint waist_roll_joint: type revolute -> fixed
- joint waist_yaw_joint: type revolute -> fixed

Commit message: 29dof_10action

File: exts/humarconoid/humarconoid/robots/G1/g1_29dof_rev_1_0.urdf (robot description, URDF)
Before this commit: robot g1_kist, 39 links, 38 joints
Joints:
- joint left_elbow_joint: type fixed -> revolute
- joint left_shoulder_pitch_joint: type fixed -> revolute
- joint left_shoulder_roll_joint: type fixed -> revolute
- joint left_shoulder_yaw_joint: type fixed -> revolute
- joint left_wrist_pitch_joint: type fixed -> revolute
- joint left_wrist_roll_joint: type fixed -> revolute
- joint left_wrist_yaw_joint: type fixed -> revolute
- joint right_elbow_joint: type fixed -> revolute
- joint right_shoulder_pitch_joint: type fixed -> revolute
- joint right_shoulder_roll_joint: type fixed -> revolute
- joint right_shoulder_yaw_joint: type fixed -> revolute
- joint right_wrist_pitch_joint: type fixed -> revolute
- joint right_wrist_roll_joint: type fixed -> revolute
- joint right_wrist_yaw_joint: type fixed -> revolute
- joint waist_pitch_joint: type fixed -> revolute
- joint waist_roll_joint: type fixed -> revolute
- joint waist_yaw_joint: type fixed -> revolute
