Commit message: reshape_rewards

File: source/humarconoid/humarconoid/robots/G1/g1_29dof_rev_1_0.urdf (robot description, URDF)
Before this commit: robot g1_kist, 39 links, 38 joints
Joints:
- joint left_elbow_joint: type revolute -> fixed
- joint left_shoulder_pitch_joint: type revolute -> fixed
- joint left_shoulder_roll_joint: type revolute -> fixed
- joint left_shoulder_yaw_joint: type revolute -> fixed
- joint left_wrist_pitch_joint: type revolute -> fixed
- joint left_wrist_roll_joint: type revolute -> fixed
- joint left_wrist_yaw_joint: type revolute -> fixed
- joint right_elbow_joint: type revolute -> fixed
- joint right_shoulder_pitch_joint: type revolute -> fixed
- joint right_shoulder_roll_joint: type revolute -> fixed
- joint right_shoulder_yaw_joint: type revolute -> fixed
- joint right_wrist_pitch_joint: type revolute -> fixed
- joint right_wrist_roll_joint: type revolute -> fixed
- joint right_wrist_yaw_joint: type revolute -> fixed
- joint waist_pitch_joint: type revolute -> fixed
- joint waist_roll_joint: type revolute -> fixed
- joint waist_yaw_joint: type revolute -> fixed
