Commit message: 2025-05-26_16-01-46

File: source/humarconoid/humarconoid/robots/G1/g1_29dof_rev_1_00.urdf (robot description, URDF)
Before this commit: robot g1_kist, 39 links, 38 joints
Links:
- link left_ankle_roll_link: geometry collision box size=0.207 0.06 0.01; visual mesh filename=meshes_kist/left_ankle_roll_link.STL
- link right_ankle_roll_link: geometry collision box size=0.207 0.06 0.01; visual mesh filename=meshes_kist/right_ankle_roll_link.STL
